File: Adapter-CMRI8-3dot5mm-adapter.brd (EAGLE design)
At the start: 31 x 50 mm, 15 parts, among them M1 MOUNTINGHOLE, M2 MOUNTINGHOLE

Commit message: initial version
converted from Plocher's RJ45 board
Parts:
- added U$2: (no value), MRCSLogoBtm:MRCSLOGOBTM
Other:
- board text added: "8 pin Molex to 3.5mm"
- board text added: "Seth Neumann John Plocher"
- board text removed: "Frog Pwr"
- board text removed: "Go Bears!"
- board text removed: "MRCS"
- board text removed: "RJ45"
- board text removed: "SPCoast"
- board text removed: "Tie points"
- board text removed: "no nc C"
- board text removed: "www . SPCoast . com"
